File: pcb/dekatron.kicad_sch (KiCad schematic)
At the start: 73 parts, among them J1 USB_C_Receptacle_USB2.0, J2 Conn_01x05, Q1 MMBTA42, Q2 S8050_SOT23, Q3 MMBTA42, Q4 IPN70R750P7S, Q5 MMBTA92, SW1 SW_Push, U1 ESP32-C3-WROOM-02, U2 MT2492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

Commit message: Write readme
Other:
- note added: "D8 green D9 red"
Changed lines of the file:
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@@
     (stroke (width 0) (type default))
+  )
+  (text "D8 green\nD9 red" (at 25.4 229.235 0)
+    (effects (font (size 1.27 1.27)) (justify left bottom))
   )
   (text "Is 12V needed, or can we use 5V?\nNo, 5V doesn't work in original."
